Commit message: move ur description to inside package folder and add functions for finding, updating urdf

File: src/rerun_rlds_ur5/ur_description/ur5_updated.urdf (robot description, URDF)
Before this commit: robot ur5_robot, 11 links, 10 joints
Links:
- link base_link_inertia: geometry collision mesh filename=/home/will/workspace/rerun_rlds_ur5/src/rerun_rlds_ur5/ur_d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; visual mesh filename=/home/will/workspace/rerun_rlds_ur5/src/rerun_rlds_ur5/ur_d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
- link forearm_link: geometry collision mesh filename=/home/will/workspace/rerun_rlds_ur5/src/rerun_rlds_ur5/ur_d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; visual mesh filename=/home/will/workspace/rerun_rlds_ur5/src/rerun_rlds_ur5/ur_d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
- link shoulder_link: geometry collision mesh filename=/home/will/workspace/rerun_rlds_ur5/src/rerun_rlds_ur5/ur_d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; visual mesh filename=/home/will/workspace/rerun_rlds_ur5/src/rerun_rlds_ur5/ur_d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
- link upper_arm_link: geometry collision mesh filename=/home/will/workspace/rerun_rlds_ur5/src/rerun_rlds_ur5/ur_d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; visual mesh filename=/home/will/workspace/rerun_rlds_ur5/src/rerun_rlds_ur5/ur_d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
- link wrist_1_link: geometry collision mesh filename=/home/will/workspace/rerun_rlds_ur5/src/rerun_rlds_ur5/ur_d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; visual mesh filename=/home/will/workspace/rerun_rlds_ur5/src/rerun_rlds_ur5/ur_d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
- link wrist_2_link: geometry collision mesh filename=/home/will/workspace/rerun_rlds_ur5/src/rerun_rlds_ur5/ur_d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; visual mesh filename=/home/will/workspace/rerun_rlds_ur5/src/rerun_rlds_ur5/ur_d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
- link wrist_3_link: geometry collision mesh filename=/home/will/workspace/rerun_rlds_ur5/src/rerun_rlds_ur5/ur_d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; visual mesh filename=/home/will/workspace/rerun_rlds_ur5/src/rerun_rlds_ur5/ur_d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
